Commit message: Add depthcam and ray sensors

File: urdf/iris/iris_14ranges.xacro (robot description, xacro)
@@ -7,8 +7,9 @@
     max="6.0"
     min="0.01"
-    step_x1="0.10"
-    step_x2="0.09"
-    step_z1="0.05"
-    step_z2="0.04"
+    offX_front="0.10"
+    offX_back="-0.09"
+    offZ_up="0.05"
+    offZ_horizon1="0.05"
+    offZ_down="-0.04"
   />
 </robot>

File: urdf/iris/iris_depthcam.xacro (robot description, xacro)
@@ -5,18 +5,21 @@
   <xacro:include filename="$(find mav_tunnel_nav)/urdf/parts/depthcam/depthcam.urdf.xacro" />
   <xacro:depth_camera
-    name="camera" parent="${namespace}/base_link" ros_topic="depthcam"
-    update_rate="20" min_range="0" max_range="3"
-    field_of_view="2" ray_count="1">
-    <origin xyz="0 0 0.036" rpy="0 0 0" />
+    name="camera" parent_link="${namespace}/base_link"
+    update_rate="20" min_range="0.05" max_range="3" field_of_view="1.047198">
+    <origin xyz="0.03 0 0.07" rpy="0 0 0" />
   </xacro:depth_camera>
   <!-- ray sensors -->
-  <!-- <xacro:include filename="$(find mav_tunnel_nav)/urdf/parts/range/range1ray_14align.urdf.xacro" />
+  <xacro:include filename="$(find mav_tunnel_nav)/urdf/parts/range/range1ray_14align.urdf.xacro" />
   <xacro:range1ray_14align_macro
-    max="6.0"
+    max="1.5"
     min="0.01"
-    step_x1="0.10"
-    step_x2="0.09"
-    step_z1="0.05"
-    step_z2="0.04"
-  /> -->
+    offX_front="0.11"
+    offX_back="-0.12"
+    offY_left="0.06"
+    offY_right="-0.06"
+    offZ_up="0.09"
+    offZ_horizon1="0.04"
+    offZ_horizon2="-0.01"
+    offZ_down="-0.04"
+  />
 </robot>

File: urdf/parts/depthcam/depthcam.urdf.xacro (robot description, xacro)
@@ -4,13 +4,13 @@
 -->
 <robot xmlns:xacro="http://ros.org/wiki/xacro">
-  <xacro:macro name="depth_camera" params="name parent *origin ros_topic update_rate min_range max_range field_of_view ray_count">
+  <xacro:macro name="depth_camera" params="name parent_link *origin update_rate:=20 min_range:=0.05 max_range:=3.0 field_of_view:=1.047198">
     <joint name="${name}_joint" type="fixed">
       <xacro:insert_block name="origin" />
-      <parent link="${parent}"/>
-      <child link="${name}_link"/>
+      <parent link="${parent_link}"/>
+      <child link="${namespace}/${name}_link"/>
     </joint>
-    <link name="${name}_link">
+    <link name="${namespace}/${name}_link">
       <inertial>
-        <mass value="0.001" />
+        <mass value="0.1" />
         <origin xyz="0 0 0" rpy="0 0 0" />
         <inertia ixx="0.000000017" ixy="0" ixz="0" iyy="0.000000017" iyz="0" izz="0.000000017" />
@@ -19,19 +19,19 @@
         <origin xyz="0 0 0" rpy="0 0 0" />
         <geometry>
-          <box size="0.073000 0.276000 0.072000" />
+          <mesh filename="model://kinect/meshes/kinect.dae" />
         </geometry>
       </visual>
       <collision>
-        <origin xyz="0 0 0" rpy="0 0 0" />
+        <origin xyz="-0.033000 0 0" rpy="0 0 0" />
         <geometry>
-          <box size="0.073000 0.276000 0.072000" />
+          <box size="0.067000 0.276000 0.036000" />
         </geometry>
       </collision>
     </link>
-    <gazebo reference="${name}_link">
+    <gazebo reference="${namespace}/${name}_link">
       <sensor name="camera" type="depth">
-        <update_rate>20</update_rate>
+        <update_rate>${update_rate}</update_rate>
         <camera>
-          <horizontal_fov>1.047198</horizontal_fov>
+          <horizontal_fov>${field_of_view}</horizontal_fov>
           <image>
             <width>640</width>
@@ -40,6 +40,6 @@
           </image>
           <clip>
-            <near>0.05</near>
-            <far>3</far>
+            <near>${min_range}</near>
+            <far>${max_range}</far>
           </clip>
         </camera>
@@ -50,11 +50,11 @@
             will control the frame rate. -->
           <updateRate>0.0</updateRate>
-          <cameraName>camera_ir</cameraName>
-          <imageTopicName>/camera/depth/image_raw</imageTopicName>
-          <cameraInfoTopicName>/camera/depth/camera_info</cameraInfoTopicName>
-          <depthImageTopicName>/camera/depth/image_raw</depthImageTopicName>
-          <depthImageInfoTopicName>/camera/depth/camera_info</depthImageInfoTopicName>
-          <pointCloudTopicName>/camera/depth/points</pointCloudTopicName>
-          <frameName>camera_link</frameName>
+          <cameraName>${name}_ir</cameraName>
+          <imageTopicName>${name}/depth/image_raw</imageTopicName>
+          <cameraInfoTopicName>${name}/depth/camera_info</cameraInfoTopicName>
+          <depthImageTopicName>${name}/depth/image_raw</depthImageTopicName>
+          <depthImageInfoTopicName>${name}/depth/camera_info</depthImageInfoTopicName>
+          <pointCloudTopicName>${name}/depth/points</pointCloudTopicName>
+          <frameName>${name}_link</frameName>
           <pointCloudCutoff>0.05</pointCloudCutoff>
           <distortionK1>0</distortionK1>

File: urdf/parts/range/range1ray.urdf.xacro (robot description, xacro)
@@ -23,10 +23,10 @@
         </geometry>
       </visual>
-      <collision>
+      <!-- <collision>
         <origin xyz="0 0 0" rpy="0 0 0" />
         <geometry>
           <box size="0.01 0.01 0.01" />
         </geometry>
-      </collision>
+      </collision> -->
     </link>
     <gazebo reference="${name}_link">

File: urdf/parts/range/range1ray_14align.urdf.xacro (robot description, xacro)
@@ -1,5 +1,5 @@
 <?xml version="1.0"?>
 <robot name="quadrotor" xmlns:xacro="http://www.ros.org/wiki/xacro">
-    <xacro:macro name="range1ray_14align_macro" params="rate:=10 min:=0.01 max:=10.0 ray_fov:=3 step_x1:=0.05 step_x2:=0.05 step_y1:=0.05 step_y2:=0.05 step_z1=0.05 step_z2=0.05 parent_link:=${namespace}/base_link">
+    <xacro:macro name="range1ray_14align_macro" params="rate:=10 min:=0.01 max:=10.0 ray_fov:=3 offX_front:=0.05 offX_back:=-0.05 offY_left:=0.05 offY_right:=-0.05 offZ_up:=0.05 offZ_horizon1:=0.05 offZ_horizon2:=0.05 offZ_down:=-0.05 parent_link:=${namespace}/base_link">
       <xacro:property name="M_PI" value="3.1415926535897932" />
       <!-- ray sensors -->
@@ -7,57 +7,57 @@
       <!-- front -->
       <xacro:sonar_sensor name="ray_front" parent="${parent_link}" ros_topic="range_front" update_rate="${rate}" min_range="${min}" max_range="${max}" field_of_view="${ray_fov*M_PI/180}" ray_count="1">
-        <origin xyz="${step_x1} 0.0 ${step_z1}" rpy="0 0 0" />
+        <origin xyz="${offX_front} 0.0 ${offZ_horizon1}" rpy="0 0 0" />
       </xacro:sonar_sensor>
       <!-- right front -->
       <xacro:sonar_sensor name="ray_rfront" parent="${parent_link}" ros_topic="range_rfront" update_rate="${rate}" min_range="${min}" max_range="${max}" field_of_view="${ray_fov*M_PI/180}" ray_count="1">
-        <origin xyz="${step_x1} ${-step_y2} ${step_z1}" rpy="0 0 ${-45*M_PI/180}" />
+        <origin xyz="${offX_front} ${offY_right} ${offZ_horizon1}" rpy="0 0 ${-45*M_PI/180}" />
       </xacro:sonar_sensor>
       <!-- left front -->
       <xacro:sonar_sensor name="ray_lfront" parent="${parent_link}" ros_topic="range_lfront" update_rate="${rate}" min_range="${min}" max_range="${max}" field_of_view="${ray_fov*M_PI/180}" ray_count="1">
-        <origin xyz="${step_x1} ${step_y1} ${step_z1}" rpy="0 0 ${45*M_PI/180}" />
+        <origin xyz="${offX_front} ${offY_left} ${offZ_horizon1}" rpy="0 0 ${45*M_PI/180}" />
       </xacro:sonar_sensor>
       <!-- right -->
       <xacro:sonar_sensor name="ray_right" parent="${parent_link}" ros_topic="range_right" update_rate="${rate}" min_range="${min}" max_range="${max}" field_of_view="${ray_fov*M_PI/180}" ray_count="1">
-        <origin xyz="0 ${-step_y2} ${step_z1}" rpy="0 0 ${-90*M_PI/180}" />
+        <origin xyz="0 ${offY_right} ${offZ_horizon2}" rpy="0 0 ${-90*M_PI/180}" />
       </xacro:sonar_sensor>
       <!-- left -->
       <xacro:sonar_sensor name="ray_left" parent="${parent_link}" ros_topic="range_left" update_rate="${rate}" min_range="${min}" max_range="${max}" field_of_view="${ray_fov*M_PI/180}" ray_count="1">
-        <origin xyz="0 ${step_y1} ${step_z1}" rpy="0 0 ${90*M_PI/180}" />
+        <origin xyz="0 ${offY_left} ${offZ_horizon2}" rpy="0 0 ${90*M_PI/180}" />
       </xacro:sonar_sensor>
       <!-- right rear -->
       <xacro:sonar_sensor name="ray_rrear" parent="${parent_link}" ros_topic="range_rrear" update_rate="${rate}" min_range="${min}" max_range="${max}" field_of_view="${ray_fov*M_PI/180}" ray_count="1">
-        <origin xyz="${-step_x2} ${-step_y2} ${step_z1}" rpy="0 0 ${-135*M_PI/180}" />
+        <origin xyz="${offX_back} ${offY_right} ${offZ_horizon1}" rpy="0 0 ${-135*M_PI/180}" />
       </xacro:sonar_sensor>
       <!-- left rear -->
       <xacro:sonar_sensor name="ray_lrear" parent="${parent_link}" ros_topic="range_lrear" update_rate="${rate}" min_range="${min}" max_range="${max}" field_of_view="${ray_fov*M_PI/180}" ray_count="1">
-        <origin xyz="${-step_x2} ${step_y1} ${step_z1}" rpy="0 0 ${135*M_PI/180}" />
+        <origin xyz="${offX_back} ${offY_left} ${offZ_horizon1}" rpy="0 0 ${135*M_PI/180}" />
       </xacro:sonar_sensor>
       <!-- rear -->
       <xacro:sonar_sensor name="ray_rear" parent="${parent_link}" ros_topic="range_rear" update_rate="${rate}" min_range="${min}" max_range="${max}" field_of_view="${ray_fov*M_PI/180}" ray_count="1">
-        <origin xyz="${-step_x2} 0 ${step_z1}" rpy="0 0 ${-180*M_PI/180}" />
+        <origin xyz="${offX_back} 0 ${offZ_horizon1}" rpy="0 0 ${-180*M_PI/180}" />
       </xacro:sonar_sensor>
       <!-- upward -->
       <xacro:sonar_sensor name="ray_up" parent="${parent_link}" ros_topic="range_up" update_rate="${rate}" min_range="${min}" max_range="${max}" field_of_view="${ray_fov*M_PI/180}" ray_count="1">
-        <origin xyz="0 0 ${step_z1}" rpy="0 ${-90*M_PI/180} 0" />
+        <origin xyz="0 0 ${offZ_up}" rpy="0 ${-90*M_PI/180} 0" />
       </xacro:sonar_sensor>
       <!-- up front -->
       <xacro:sonar_sensor name="ray_ufront" parent="${parent_link}" ros_topic="range_ufront" update_rate="${rate}" min_range="${min}" max_range="${max}" field_of_view="${ray_fov*M_PI/180}" ray_count="1">
-        <origin xyz="${step_x1/3} 0 ${step_z1}" rpy="0 ${-45*M_PI/180} 0" />
+        <origin xyz="${offX_front/3} 0 ${offZ_up}" rpy="0 ${-45*M_PI/180} 0" />
       </xacro:sonar_sensor>
       <!-- up rear -->
       <xacro:sonar_sensor name="ray_urear" parent="${parent_link}" ros_topic="range_urear" update_rate="${rate}" min_range="${min}" max_range="${max}" field_of_view="${ray_fov*M_PI/180}" ray_count="1">
-        <origin xyz="${-step_x2/3} 0 ${step_z1}" rpy="0 ${-45*M_PI/180} ${180*M_PI/180}" />
+        <origin xyz="${offX_back/3} 0 ${offZ_up}" rpy="0 ${-45*M_PI/180} ${180*M_PI/180}" />
       </xacro:sonar_sensor>
       <!-- downward -->
       <xacro:sonar_sensor name="ray_down" parent="${parent_link}" ros_topic="range_down" update_rate="${rate}" min_range="${min}" max_range="${max}" field_of_view="${ray_fov*M_PI/180}" ray_count="1">
-        <origin xyz="0 0 ${-step_z2}" rpy="0 ${90*M_PI/180} 0" />
+        <origin xyz="0 0 ${offZ_down}" rpy="0 ${90*M_PI/180} 0" />
       </xacro:sonar_sensor>
       <!-- down front -->
       <xacro:sonar_sensor name="ray_dfront" parent="${parent_link}" ros_topic="range_dfront" update_rate="${rate}" min_range="${min}" max_range="${max}" field_of_view="${ray_fov*M_PI/180}" ray_count="1">
-        <origin xyz="${step_x1/3} 0 ${-step_z2}" rpy="0 ${45*M_PI/180} 0" />
+        <origin xyz="${offX_front/3} 0 ${offZ_down}" rpy="0 ${45*M_PI/180} 0" />
       </xacro:sonar_sensor>
       <!-- down rear -->
       <xacro:sonar_sensor name="ray_drear" parent="${parent_link}" ros_topic="range_drear" update_rate="${rate}" min_range="${min}" max_range="${max}" field_of_view="${ray_fov*M_PI/180}" ray_count="1">
-        <origin xyz="${-step_x2/3} 0 ${-step_z2}" rpy="0 ${45*M_PI/180} ${180*M_PI/180}" />
+        <origin xyz="${offX_back/3} 0 ${offZ_down}" rpy="0 ${45*M_PI/180} ${180*M_PI/180}" />
       </xacro:sonar_sensor>
     </xacro:macro>
