Commit message: Add description of depthcam (incomplete)

File: urdf/iris/iris_depthcam.xacro (robot description, xacro)
@@ -3,4 +3,11 @@
   <xacro:include filename="$(find mav_tunnel_nav)/urdf/parts/rotors_custom/iris_base.xacro" />
   <!-- depth camera -->
+  <xacro:include filename="$(find mav_tunnel_nav)/urdf/parts/depthcam/depthcam.urdf.xacro" />
+  <xacro:depth_camera
+    name="camera" parent="${namespace}/base_link" ros_topic="depthcam"
+    update_rate="20" min_range="0" max_range="3"
+    field_of_view="2" ray_count="1">
+    <origin xyz="0 0 0.036" rpy="0 0 0" />
+  </xacro:depth_camera>
   <!-- ray sensors -->
   <!-- <xacro:include filename="$(find mav_tunnel_nav)/urdf/parts/range/range1ray_14align.urdf.xacro" />

File: urdf/parts/depthcam/depthcam.urdf.xacro (robot description, xacro)
@@ -4,5 +4,5 @@
 -->
 <robot xmlns:xacro="http://ros.org/wiki/xacro">
-  <!-- <xacro:macro name="sonar_sensor" params="name parent *origin ros_topic update_rate min_range max_range field_of_view ray_count">
+  <xacro:macro name="depth_camera" params="name parent *origin ros_topic update_rate min_range max_range field_of_view ray_count">
     <joint name="${name}_joint" type="fixed">
       <xacro:insert_block name="origin" />
@@ -19,5 +19,5 @@
         <origin xyz="0 0 0" rpy="0 0 0" />
         <geometry>
-          <box size="0.01 0.01 0.01" />
+          <box size="0.073000 0.276000 0.072000" />
         </geometry>
       </visual>
@@ -25,45 +25,50 @@
         <origin xyz="0 0 0" rpy="0 0 0" />
         <geometry>
-          <box size="0.01 0.01 0.01" />
+          <box size="0.073000 0.276000 0.072000" />
         </geometry>
       </collision>
     </link>
     <gazebo reference="${name}_link">
-      <sensor type="ray" name="${name}">
-        <pose>0 0 0 0 0 0</pose>
-        <visualize>true</visualize>
-        <update_rate>${update_rate}</update_rate>
-        <ray>
-          <scan>
-            <horizontal>
-              <samples>${ray_count}</samples>
-              <resolution>1</resolution>
-              <min_angle>-${field_of_view/2}</min_angle>
-              <max_angle> ${field_of_view/2}</max_angle>
-            </horizontal>
-            <vertical>
-              <samples>${ray_count}</samples>
-              <resolution>1</resolution>
-              <min_angle>-${field_of_view/2}</min_angle>
-              <max_angle> ${field_of_view/2}</max_angle>
-            </vertical>
-          </scan>
-          <range>
-            <min>${min_range}</min>
-            <max>${max_range}</max>
-            <resolution>0.01</resolution>
-          </range>
-        </ray>
-        <plugin filename="libgazebo_ros_range.so" name="gazebo_ros_range">
-          <gaussianNoise>0.005</gaussianNoise>
+      <sensor name="camera" type="depth">
+        <update_rate>20</update_rate>
+        <camera>
+          <horizontal_fov>1.047198</horizontal_fov>
+          <image>
+            <width>640</width>
+            <height>480</height>
+            <format>R8G8B8</format>
+          </image>
+          <clip>
+            <near>0.05</near>
+            <far>3</far>
+          </clip>
+        </camera>
+        <plugin name="camera_plugin" filename="libgazebo_ros_openni_kinect.so">
+          <baseline>0.2</baseline>
           <alwaysOn>true</alwaysOn>
-          <updateRate>${update_rate}</updateRate>
-          <topicName>${ros_topic}</topicName>
-          <frameName>${name}_link</frameName>
-          <radiation>infrared</radiation>
-          <fov>${field_of_view}</fov>
+          <!-- Keep this zero, update_rate in the parent <sensor> tag
+            will control the frame rate. -->
+          <updateRate>0.0</updateRate>
+          <cameraName>camera_ir</cameraName>
+          <imageTopicName>/camera/depth/image_raw</imageTopicName>
+          <cameraInfoTopicName>/camera/depth/camera_info</cameraInfoTopicName>
+          <depthImageTopicName>/camera/depth/image_raw</depthImageTopicName>
+          <depthImageInfoTopicName>/camera/depth/camera_info</depthImageInfoTopicName>
+          <pointCloudTopicName>/camera/depth/points</pointCloudTopicName>
+          <frameName>camera_link</frameName>
+          <pointCloudCutoff>0.05</pointCloudCutoff>
+          <distortionK1>0</distortionK1>
+          <distortionK2>0</distortionK2>
+          <distortionK3>0</distortionK3>
+          <distortionT1>0</distortionT1>
+          <distortionT2>0</distortionT2>
+          <CxPrime>0</CxPrime>
+          <Cx>0</Cx>
+          <Cy>0</Cy>
+          <focalLength>0</focalLength>
+          <hackBaseline>0</hackBaseline>
         </plugin>
       </sensor>
     </gazebo>
-  </xacro:macro> -->
+  </xacro:macro>
 </robot>

Commit message: Realign sensors

File: urdf/iris/iris_depthcam.xacro (robot description, xacro)
@@ -7,5 +7,5 @@
     name="camera" parent_link="${namespace}/base_link"
     update_rate="20" min_range="0.05" max_range="3" field_of_view="1.047198">
-    <origin xyz="0.03 0 0.07" rpy="0 0 0" />
+    <origin xyz="0.03 0 -0.06" rpy="0 0 0" />
   </xacro:depth_camera>
   <!-- ray sensors -->
@@ -18,8 +18,8 @@
     offY_left="0.06"
     offY_right="-0.06"
-    offZ_up="0.09"
-    offZ_horizon1="0.04"
-    offZ_horizon2="-0.01"
-    offZ_down="-0.04"
+    offZ_up="0.055"
+    offZ_horizon1="-0.01"
+    offZ_horizon2="0.01"
+    offZ_down="-0.085"
   />
 </robot>

Commit message: Reconfigure depth cam

File: urdf/iris/iris_depthcam.xacro (robot description, xacro)
@@ -6,5 +6,5 @@
   <xacro:depth_camera
     name="camera" parent_link="${namespace}/base_link"
-    update_rate="20" min_range="0.05" max_range="3" field_of_view="1.047198">
+    update_rate="20" min_range="0.05" max_range="30" field_of_view="1.047198">
     <origin xyz="0.03 0 -0.06" rpy="0 0 0" />
   </xacro:depth_camera>

File: urdf/parts/depthcam/depthcam.urdf.xacro (robot description, xacro)
@@ -4,5 +4,5 @@
 -->
 <robot xmlns:xacro="http://ros.org/wiki/xacro">
-  <xacro:macro name="depth_camera" params="name parent_link *origin update_rate:=20 min_range:=0.05 max_range:=3.0 field_of_view:=1.047198">
+  <xacro:macro name="depth_camera" params="name parent_link *origin update_rate:=20 min_range:=0.05 max_range:=3.0 field_of_view:=1.3671">
     <joint name="${name}_joint" type="fixed">
       <xacro:insert_block name="origin" />
@@ -12,5 +12,5 @@
     <link name="${namespace}/${name}_link">
       <inertial>
-        <mass value="0.1" />
+        <mass value="0.01" />
         <origin xyz="0 0 0" rpy="0 0 0" />
         <inertia ixx="0.000000017" ixy="0" ixz="0" iyy="0.000000017" iyz="0" izz="0.000000017" />
@@ -41,5 +41,5 @@
           <horizontal_fov>${field_of_view}</horizontal_fov>
           <image>
-            <width>640</width>
+            <width>752</width>
             <height>480</height>
             <format>R8G8B8</format>

Commit message: Add fisheye

File: urdf/iris/iris_depthcam.xacro (robot description, xacro)
@@ -6,7 +6,14 @@
   <xacro:depth_camera
     name="camera" parent_link="${namespace}/base_link"
-    update_rate="20" min_range="0.05" max_range="30" field_of_view="1.047198">
-    <origin xyz="0.03 0 -0.06" rpy="0 0 0" />
+    update_rate="20" min_range="0.05" max_range="10" field_of_view="1.047198">
+    <origin xyz="0.00 0 -0.06" rpy="0 0 0" />
   </xacro:depth_camera>
+  <!-- fisheye cam -->
+  <xacro:include filename="$(find mav_tunnel_nav)/urdf/parts/fisheye/fisheye.urdf.xacro" />
+  <xacro:fisheye_camera
+    name="camera" parent_link="${namespace}/base_link"
+    update_rate="20" min_range="0.05" max_range="30.0" field_of_view="2.84489">
+    <origin xyz="0.11 0 0.03" rpy="0 0 0" />
+  </xacro:fisheye_camera>
   <!-- ray sensors -->
   <xacro:include filename="$(find mav_tunnel_nav)/urdf/parts/range/range1ray_14align.urdf.xacro" />

Commit message: Flashlight in a dark cave

File: urdf/iris/iris_depthcam.xacro (robot description, xacro)
@@ -23,3 +23,56 @@
     offZ_down="-0.085"
   />
+  <!-- flashlight -->
+  <gazebo>
+    <model name='flashlight'>
+      <pose>0.1 0 0.05 0 -1.57 0</pose>
+      <link name='light_source'>
+        <inertial>
+          <mass>0.00001</mass>
+          <inertia>
+            <ixx>1.0e-05</ixx>
+            <ixy>0</ixy>
+            <ixz>0</ixz>
+            <iyy>1.0e-05</iyy>
+            <iyz>0</iyz>
+            <izz>1.0e-05</izz>
+          </inertia>
+        </inertial>
+        <light name='lamp_light' type='spot'>
+          <attenuation>
+            <range>50</range>
+            <linear>0.05</linear>
+          </attenuation>
+          <diffuse>1 1 1 1</diffuse>
+          <specular>1 1 1 1</specular>
+          <spot>
+            <inner_angle>1</inner_angle>
+            <outer_angle>1.1</outer_angle>
+            <falloff>1</falloff>
+          </spot>
+          <direction>0 0 -1</direction>
+        </light>
+        <visual name='lamp'>
+          <geometry>
+            <sphere>
+              <radius>0.010</radius>
+            </sphere>
+          </geometry>
+          <transparency>0</transparency>
+          <material>
+            <ambient>1 1 1 1</ambient>
+            <diffuse>1 1 1 1</diffuse>
+            <specular>1 1 1 1</specular>
+            <emissive>1 1 1 1</emissive>
+          </material>
+        </visual>
+      </link>
+    </model>
+  </gazebo>
+  <gazebo>
+    <joint name='flashlight_joint' type='fixed'>
+      <parent>${namespace}/base_link</parent>
+      <child>flashlight::light_source</child>
+    </joint>
+  </gazebo>
 </robot>

Commit message: configuration for textured cave

File: urdf/iris/iris_depthcam.xacro (robot description, xacro)
@@ -47,6 +47,6 @@
           <specular>1 1 1 1</specular>
           <spot>
-            <inner_angle>1</inner_angle>
-            <outer_angle>1.1</outer_angle>
+            <inner_angle>1.1</inner_angle>
+            <outer_angle>1.2</outer_angle>
             <falloff>1</falloff>
           </spot>

File: urdf/parts/depthcam/depthcam.urdf.xacro (robot description, xacro)
@@ -12,6 +12,6 @@
     <link name="${namespace}/${name}_link">
       <inertial>
-        <mass value="0.01" />
-        <origin xyz="0 0 0" rpy="0 0 0" />
+        <mass value="0.005" />
+        <origin xyz="-0.033000 0 0" rpy="0 0 0" />
         <inertia ixx="0.000000017" ixy="0" ixz="0" iyy="0.000000017" iyz="0" izz="0.000000017" />
       </inertial>
