Commit message: urdf: make sonar frame under each robot

File: urdf/parts/range/range1ray.urdf.xacro (robot description, xacro)
@@ -9,7 +9,7 @@
       <xacro:insert_block name="origin" />
       <parent link="${parent}"/>
-      <child link="${name}_link"/>
+      <child link="${namespace}/${name}_link"/>
     </joint>
-    <link name="${name}_link">
+    <link name="${namespace}/${name}_link">
       <inertial>
         <mass value="0.001" />
@@ -30,5 +30,5 @@
       </collision> -->
     </link>
-    <gazebo reference="${name}_link">
+    <gazebo reference="${namespace}/${name}_link">
       <sensor type="ray" name="${name}">
         <pose>0 0 0 0 0 0</pose>
@@ -61,5 +61,5 @@
           <updateRate>${update_rate}</updateRate>
           <topicName>${ros_topic}</topicName>
-          <frameName>${name}_link</frameName>
+          <frameName>${namespace}/${name}_link</frameName>
           <radiation>infrared</radiation>
           <fov>${field_of_view}</fov>
