Commit message: Replace depth camera's model

File: urdf/parts/depthcam/depthcam.urdf.xacro (robot description, xacro)
@@ -17,7 +17,13 @@
       </inertial>
       <visual>
+        <!--
         <origin xyz="0 0 0" rpy="0 0 0" />
         <geometry>
           <mesh filename="model://kinect/meshes/kinect.dae" />
+        </geometry>
+        -->
+        <origin xyz="-0.033000 0 0" rpy="0 0 0" />
+        <geometry>
+          <box size="0.067000 0.276000 0.036000" />
         </geometry>
       </visual>

Commit message: urdf: adjust depth camp freq etc

File: urdf/parts/depthcam/depthcam.urdf.xacro (robot description, xacro)
@@ -4,5 +4,5 @@
 -->
 <robot xmlns:xacro="http://ros.org/wiki/xacro">
-  <xacro:macro name="depth_camera" params="name parent_link *origin update_rate:=20 min_range:=0.05 max_range:=3.0 field_of_view:=1.3671">
+  <xacro:macro name="depth_camera" params="name parent_link *origin update_rate:=5 min_range:=0.05 max_range:=3.0 field_of_view:=1.3671">
     <joint name="${name}_joint" type="fixed">
       <xacro:insert_block name="origin" />

File: urdf/parts/rotors_custom/iris_base.xacro (robot description, xacro)
@@ -6,8 +6,4 @@
   <!-- Instantiate a controller. -->
   <xacro:controller_plugin_macro namespace="${namespace}" imu_sub_topic="imu" />
-  <xacro:if value="$(arg enable_mavlink_interface)">
-    <!-- Instantiate mavlink telemetry interface. -->
-    <xacro:default_mavlink_interface namespace="${namespace}" imu_sub_topic="imu" rotor_count="4" />
-  </xacro:if>
   <!-- Mount an ADIS16448 IMU. -->
   <!--<xacro:default_imu namespace="${namespace}" parent_link="${namespace}/base_link" />-->
@@ -46,14 +42,3 @@
     <origin xyz="0.0 0.0 0.0" rpy="0.0 0.0 0.0" />
   </xacro:odometry_plugin_macro>
-  <xacro:if value="$(arg enable_ground_truth)">
-    <xacro:ground_truth_imu_and_odometry namespace="${namespace}" parent_link="${namespace}/base_link" />
-  </xacro:if>
-  <xacro:if value="$(arg enable_logging)">
-    <!-- Instantiate a logger -->
-    <xacro:bag_plugin_macro
-      namespace="${namespace}"
-      bag_file="$(arg log_file)"
-      rotor_velocity_slowdown_sim="${rotor_velocity_slowdown_sim}"
-      wait_to_record_bag="$(arg wait_to_record_bag)" />
-  </xacro:if>
 </robot>
